Commit message: gripper end effector

File: src/abb_irb120_description/urdf/irb120_3_60.xacro (robot description, xacro)
@@ -2,4 +2,11 @@
 <robot name="abb_irb120_3_60" xmlns:xacro="http://ros.org/wiki/xacro">
   <xacro:include filename="$(find abb_irb120_description)/urdf/irb120_3_60_macro.xacro"/>
+  <xacro:include filename="$(find abb_irb120_description)/urdf/gripper_macro.xacro"/>
   <xacro:abb_irb120_3_60 prefix=""/>
+  <xacro:gripper prefix=""/>
+  <joint name="tool0-gripper_base" type="fixed">
+    <parent link="tool0"/>
+    <child link="gripper_base"/>
+    <origin xyz="0 0 0" rpy="0 0 0"/>
+  </joint>
 </robot>

File: src/abb_irb120_moveit/config/abb_irb120_3_60.ros2_control.xacro (robot description, xacro)
@@ -49,4 +49,18 @@
                 <state_interface name="velocity"/>
             </joint>
+            <joint name="left_finger_joint">
+                <command_interface name="position"/>
+                <state_interface name="position">
+                <param name="initial_value">${initial_positions['left_finger_joint']}</param>
+                </state_interface>
+                <state_interface name="velocity"/>
+            </joint>
+            <joint name="right_finger_joint">
+                <command_interface name="position"/>
+                <state_interface name="position">
+                <param name="initial_value">${initial_positions['right_finger_joint']}</param>
+                </state_interface>
+                <state_interface name="velocity"/>
+            </joint>
         </ros2_control>
         <gazebo>
